Commit message: Corregir las cotas del robot: el URDF tenia largo y ancho cruzados
El usuario midio el robot con cinta, de punta a punta y CON ORUGAS:
18 cm de frente a atras y 22 de lado a lado. El URDF ponia 0.218 x 0.185,
de la ficha publicada del RVR y declarado "NO MEDIDO": modelaba un robot
mas largo que ancho siendo al reves.

  base_length  0.218 -> 0.18
  base_width   0.185 -> 0.22

Solo cambia la caja de colision y la inercia: las ruedas usan
wheel_separation, independiente, asi que ningun frame TF se mueve y la
odometria no se toca. Verificado: el xacro compila y da 0.18 x 0.22.

Y arrastraba un error real en Nav2:

  robot_radius  0.11 -> 0.145

El 0.11 estaba etiquetado como "radio circunscrito" y es aritmetica mal
hecha. El circunscrito es sqrt(0.09^2 + 0.11^2) = 0.142 con las cotas
medidas, y 0.143 incluso con las del URDF viejo: con cualquiera de los
dos se queda corto. Un robot_radius corto hace que el planificador trace
rutas donde una ESQUINA del robot roza, y no da ningun error. Lo tapaba
el collision_monitor con sus 0.18, que es probablemente por que approach
saltaba al rodear obstaculos.

collision_monitor.yaml: corregidas las cotas de los comentarios (media
longitud 0.09, no 0.109) y anotado que la holgura depende de la
direccion -- 9.0 cm de frente, 7.0 de costado, 3.8 en esquina. La
geometria del poligono Precaucion NO se toca: es la que se probo en 4
navegaciones y cambiarla obligaria a repetirlas.

Medido: con radius 0.18 el robot NO cruza un paso de 40 cm.

File: atriz_rvr_description/urdf/rvr.urdf.xacro (robot description, xacro)
@@ -42,10 +42,29 @@
        DIMENSIONES. Todo lo geométrico se cambia SOLO aquí.
        ════════════════════════════════════════════════════════════════════════ -->
-  <!-- Chasis. Fuente: especificación publicada del Sphero RVR (218 x 185 x 114 mm).
-       📝 NO MEDIDO sobre esta unidad. Afecta a la visualización y a los costmaps
-       de Nav2 (el footprint del robot), no a la odometría. -->
-  <xacro:property name="base_length" value="0.218"/>   <!-- X, hacia delante -->
-  <xacro:property name="base_width"  value="0.185"/>   <!-- Y, hacia la izquierda -->
-  <xacro:property name="base_height" value="0.114"/>   <!-- Z -->
+  <!-- Chasis. ✅ MEDIDO sobre esta unidad por el usuario el 2026-07-31, de punta
+       a punta y CON LAS ORUGAS INCLUIDAS: 18 cm de frente a atrás, 22 cm de lado
+       a lado.
+       🔴 CORREGIDO: hasta esa fecha aquí ponía 0.218 x 0.185, de la ficha
+          publicada del RVR y sin medir. Estaban **CRUZADOS**: el modelo era más
+          largo que ancho y el robot real es al revés. Se descubrió cuando el
+          usuario dio la medida al probar un paso estrecho.
+       Consecuencias, que no son cosméticas:
+         media longitud  0.09 m  (antes 0.109)  -> fija dónde para el
+                                 collision_monitor: hueco ≈ radius − 0.09
+         media anchura   0.11 m  (antes 0.0925)
+         radio INSCRITO      0.09 m
+         radio CIRCUNSCRITO  0.142 m = √(0.09² + 0.11²)
+                             -> ES EL QUE VA EN `robot_radius` DE NAV2.
+                                Estuvo en 0.11, que no es ninguno de los dos.
+       📝 base_height sigue SIN MEDIR (ficha del RVR). Es el sospechoso número
+          uno si el mapa sale inclinado (ver el bloque del LIDAR, abajo).
+       ⚠️ SIN RESOLVER: `wheel_separation` 0.150 más `wheel_width` 0.025 dan
+          17.5 cm de oruga a oruga, pero el robot mide 22 cm. O la separación
+          está corta o el cuerpo sobresale de las orugas. Es solo visual —la
+          odometría la da el locator del RVR, no estas cotas— pero está sin
+          comprobar. -->
+  <xacro:property name="base_length" value="0.18"/>    <!-- X, hacia delante  ✅ medido -->
+  <xacro:property name="base_width"  value="0.22"/>    <!-- Y, hacia la izquierda ✅ medido -->
+  <xacro:property name="base_height" value="0.114"/>   <!-- Z  📝 ficha, sin medir -->
   <!-- Ruedas/orugas. 📝 NO MEDIDO. El RVR lleva orugas de goma sobre ruedas, así
        que "radio" es una aproximación útil para visualizar y para que

Commit message: URDF con todas las cotas medidas, y corregir la premisa de la inclinacion
Medidas por el usuario el 2026-07-31, robot apagado sobre suelo plano:

    base_length      0.18  -> 0.182   frente-atras
    base_width       0.22  -> 0.217   lado a lado
    base_height      0.114 -> 0.070   suelo a la tapa (la ficha daba 11.4)
    wheel_width      0.025 -> 0.035
    wheel_separation 0.150 -> 0.183   = 0.148 interno + 0.035 de oruga
    laser_gap        0.040 -> 0.046
    x2_height        0.041 -> 0.050
    laser_z          0.1745 -> 0.155  VALOR DIRECTO, ya no una suma

laser_z era una suma derivada que arrastraba la altura equivocada de la
ficha, asi que el plano de barrido estaba 2 cm alto. El robot ve mas
abajo de lo documentado: el limite pasa de 17.45 a 15.5 cm. Es una
traslacion pura en Z, no inclina nada y no afecta a SLAM 2D ni a Nav2.

Comprobaciones que cierran: 0.148 + 2 x 0.035 = 0.218 contra 0.217 de
ancho medido, y 7.0 + 4.6 + 5.0 = 16.6 contra los 16.5 medidos hasta el
extremo superior del LIDAR. El radio circunscrito sigue en 0.142, asi
que robot_radius 0.145 no cambia.

Y se corrige la premisa del comentario de _h_quaternion. Decia que la
inclinacion de ~8 grados era real y estaba "confirmada por tres vias
independientes". No lo eran: el arbol TF sale de esta misma linea, esta
linea del cuaternion del RVR, el cuaternion de la IMU, y el acelerometro
es el mismo chip. El usuario midio el disco del LIDAR en cuatro puntos y
sale nivelado: el robot esta horizontal y los 8 grados son un desvio de
la IMU.

El comportamiento NO se cambia. Poner roll = pitch = 0 es una linea,
pero antes hay que medir la deriva de SLAM con y sin, y comparar.

File: atriz_rvr_description/urdf/rvr.urdf.xacro (robot description, xacro)
@@ -50,21 +50,21 @@
           usuario dio la medida al probar un paso estrecho.
        Consecuencias, que no son cosméticas:
-         media longitud  0.09 m  (antes 0.109)  -> fija dónde para el
-                                 collision_monitor: hueco ≈ radius − 0.09
-         media anchura   0.11 m  (antes 0.0925)
-         radio INSCRITO      0.09 m
-         radio CIRCUNSCRITO  0.142 m = √(0.09² + 0.11²)
+         media longitud  0.091 m  -> fija dónde para el collision_monitor:
+                                     hueco ≈ radius − 0.091
+         media anchura   0.1085 m
+         radio INSCRITO      0.091 m
+         radio CIRCUNSCRITO  0.142 m = √(0.091² + 0.1085²)
                              -> ES EL QUE VA EN `robot_radius` DE NAV2.
                                 Estuvo en 0.11, que no es ninguno de los dos.
-       📝 base_height sigue SIN MEDIR (ficha del RVR). Es el sospechoso número
-          uno si el mapa sale inclinado (ver el bloque del LIDAR, abajo).
-       ⚠️ SIN RESOLVER: `wheel_separation` 0.150 más `wheel_width` 0.025 dan
-          17.5 cm de oruga a oruga, pero el robot mide 22 cm. O la separación
-          está corta o el cuerpo sobresale de las orugas. Es solo visual —la
-          odometría la da el locator del RVR, no estas cotas— pero está sin
-          comprobar. -->
-  <xacro:property name="base_length" value="0.18"/>    <!-- X, hacia delante  ✅ medido -->
-  <xacro:property name="base_width"  value="0.22"/>    <!-- Y, hacia la izquierda ✅ medido -->
-  <xacro:property name="base_height" value="0.114"/>   <!-- Z  📝 ficha, sin medir -->
+       ✅ `base_height` 0.070 también MEDIDO (2026-07-31): del suelo a la tapa
+          del RVR. La ficha decía 0.114 — **4.4 cm de más**. Sobre esa tapa hay
+          además un piso de montaje de 4.6 cm donde va el LIDAR (ver abajo).
+       ✅ RESUELTO el desajuste de las orugas: son de 3.5 cm de ancho (no 2.5) y
+          van de borde interno a borde interno a 14.8 cm, o sea 18.3 entre
+          centros. Comprobación: 14.8 + 2×3.5 = 21.8 ≈ 21.7 medidos de lado a
+          lado. Las orugas ocupan TODO el ancho del robot. -->
+  <xacro:property name="base_length" value="0.182"/>   <!-- X, frente-atrás   ✅ medido -->
+  <xacro:property name="base_width"  value="0.217"/>   <!-- Y, lado a lado    ✅ medido -->
+  <xacro:property name="base_height" value="0.070"/>   <!-- Z, suelo a la tapa ✅ medido -->
   <!-- Ruedas/orugas. 📝 NO MEDIDO. El RVR lleva orugas de goma sobre ruedas, así
        que "radio" es una aproximación útil para visualizar y para que
@@ -72,29 +72,42 @@
        IMPORTANTE: estos valores NO se usan para calcular odometría — el RVR la
        entrega ya hecha por su locator interno. Son geométricos. -->
-  <xacro:property name="wheel_radius"    value="0.032"/>
-  <xacro:property name="wheel_width"     value="0.025"/>
-  <xacro:property name="wheel_separation" value="0.150"/>  <!-- entre centros, eje Y -->
+  <xacro:property name="wheel_radius"    value="0.032"/>   <!-- 📝 SIN MEDIR, ficha -->
+  <xacro:property name="wheel_width"     value="0.035"/>   <!-- ✅ medido 2026-07-31 -->
+  <!-- ✅ 0.183 = 0.148 (borde interno a borde interno) + 0.035 (un ancho de
+       oruga) = distancia entre CENTROS. Medido el 2026-07-31.
+       Cuadra: 0.148 + 2×0.035 = 0.218 ≈ 0.217 de ancho total. -->
+  <xacro:property name="wheel_separation" value="0.183"/>  <!-- entre centros, eje Y -->
   <!-- ══ POSICIÓN DEL LIDAR ══════════════════════════════════════════════════
-       ✅ CENTRADO confirmado por el usuario el 2026-07-30: el X2 está en el
-          centro del RVR, así que x=0 e y=0.
-       🟡 ALTURA DERIVADA, no medida directamente. El usuario midió **4 cm de
-          hueco entre la tapa del RVR y la base del LIDAR**. De ahí:
-              base_height        0.114   alto del RVR (ESPECIFICACIÓN, sin medir)
-            + laser_gap          0.040   hueco medido por el usuario  ✅
-            + x2_height/2        0.0205  del apoyo al centro del disco
-            ─────────────────────────
-              laser_z            0.1745  altura del plano de barrido sobre el suelo
-       El término dudoso es `base_height`: viene de la ficha del RVR y NADIE lo
-       ha medido en esta unidad. Si el mapa sale inclinado, es el primer
-       sospechoso — mide del SUELO al centro del disco y pon el resultado
-       directamente en `laser_z`, ignorando la suma.
-       Para comparar: el valor que arrastraba el proyecto era 0.10, una
-       suposición declarada en GUIA_COMPLETA_LIDAR.md. Se queda **7.5 cm corto**.
+       ✅ TODO MEDIDO el 2026-07-31, con el robot apagado sobre suelo plano.
+           suelo → tapa del RVR                 7.0 cm   ✅
+           tapa  → base del LIDAR (piso extra)  4.6 cm   ✅
+           base del LIDAR → centro del disco    3.9 cm   (= 15.5 − 11.6)
+           ────────────────────────────────────────────
+           suelo → CENTRO DEL DISCO GIRATORIO  15.5 cm   ✅  <- `laser_z`
+           suelo → extremo superior            16.5 cm   ✅  (comprobación)
+       Comprobación cruzada: 7.0 + 4.6 + 5.0 (alto del LIDAR) = 16.6 ≈ 16.5. ✅
+       🔴 CORREGIDO: `laser_z` estuvo en 0.1745 hasta esta fecha, DERIVADO de
+          `base_height` 0.114 (ficha, mal: son 0.070) + 4.0 cm de hueco + medio
+          alto del X2. El plano de barrido está **2 cm MÁS BAJO** de lo que decía
+          el modelo.
+          Consecuencia práctica: el robot ve 2 cm más abajo de lo documentado. El
+          límite «por debajo de X el LIDAR no ve nada» pasa de 17.45 a **15.5 cm**.
+          📝 Un error en `laser_z` es una traslación pura en Z: NO inclina nada y
+             no afecta a SLAM 2D ni a Nav2, que trabajan en el plano. Afecta a la
+             visualización y a ese límite de altura.
+       ✅ CENTRADO y NIVELADO, confirmado por el usuario:
+          · x = 0, y = 0 (2026-07-30)
+          · el disco está a la MISMA altura en los cuatro puntos —delante, detrás,
+            izquierda y derecha— (2026-07-31). Es decir: **el robot está físicamente
+            horizontal**, y la inclinación de ~8° que reporta la IMU NO es real.
+            Ver la cabecera de `rvr_driver_node.py` y el manual, cap. 13.
        ═══════════════════════════════════════════════════════════════════════ -->
   <xacro:property name="laser_x"   value="0.0"/>
   <xacro:property name="laser_y"   value="0.0"/>
-  <xacro:property name="laser_gap" value="0.040"/>   <!-- ✅ medido 2026-07-30 -->
-  <xacro:property name="x2_height" value="0.041"/>   <!-- alto del X2, de su ficha -->
-  <xacro:property name="laser_z"   value="${base_height + laser_gap + x2_height/2}"/>
+  <xacro:property name="laser_gap" value="0.046"/>   <!-- tapa → base del LIDAR ✅ -->
+  <xacro:property name="x2_height" value="0.050"/>   <!-- alto del X2 ✅ medido -->
+  <!-- 🔴 VALOR DIRECTO, no la suma. La suma daba 0.1745 con una ficha
+       equivocada; esto está medido con una regla desde el suelo. -->
+  <xacro:property name="laser_z"   value="0.155"/>
   <!-- IMU. Va dentro del RVR, en su placa. 📝 NO MEDIDO; se coloca en el centro
        geométrico, que es una aproximación razonable y no afecta a la odometría

Commit message: wheel_radius 0.032 -> 0.035, medido: el modelo cierra
Ultima cota que faltaba. La ficha decia 3.2 cm y son 3.5 del suelo al
centro del eje.

Cierra el modelo por un segundo camino, independiente del ancho:

  wheel_radius 0.035 -> oruga de 0.070 de diametro
  base_height        =  0.070 (medido del suelo a la tapa)

Al ser iguales, la caja del chasis queda DEL SUELO A 7 cm, que es
exactamente como se ve el RVR: las orugas ocupan todo el alto del
lateral. Verificado sobre el xacro compilado: base_footprint ->
base_link 0.035, laser a 0.155 sobre el suelo, caja de 0.000 a 0.070.

El centrado del LIDAR queda confirmado con las cotas nuevas.

File: atriz_rvr_description/urdf/rvr.urdf.xacro (robot description, xacro)
@@ -67,10 +67,15 @@
   <xacro:property name="base_width"  value="0.217"/>   <!-- Y, lado a lado    ✅ medido -->
   <xacro:property name="base_height" value="0.070"/>   <!-- Z, suelo a la tapa ✅ medido -->
-  <!-- Ruedas/orugas. 📝 NO MEDIDO. El RVR lleva orugas de goma sobre ruedas, así
-       que "radio" es una aproximación útil para visualizar y para que
-       base_footprint quede a la altura correcta.
+  <!-- Ruedas/orugas. ✅ TODO MEDIDO el 2026-07-31. El RVR lleva orugas de goma
+       sobre ruedas, así que "radio" es la distancia del suelo al centro del eje.
+       ✅ COMPROBACIÓN QUE CIERRA EL MODELO:
+            wheel_radius 0.035 → oruga de 0.070 de diámetro
+            base_height             = 0.070
+          Son iguales, así que la caja del chasis va **del suelo a 7 cm**, que es
+          exactamente como se ve el RVR: las orugas ocupan todo el alto del
+          lateral. El modelo cuadra por dos caminos distintos.
        IMPORTANTE: estos valores NO se usan para calcular odometría — el RVR la
        entrega ya hecha por su locator interno. Son geométricos. -->
-  <xacro:property name="wheel_radius"    value="0.032"/>   <!-- 📝 SIN MEDIR, ficha -->
+  <xacro:property name="wheel_radius"    value="0.035"/>   <!-- ✅ medido 2026-07-31 -->
   <xacro:property name="wheel_width"     value="0.035"/>   <!-- ✅ medido 2026-07-31 -->
   <!-- ✅ 0.183 = 0.148 (borde interno a borde interno) + 0.035 (un ancho de

Commit message: El LIDAR no estaba centrado: laser_x = -0.005, medido con cinta
El usuario midio el 2026-08-02 y el modelo estaba mal:

    chasis 19.0 cm frente-atras (con orugas)  -> centro geometrico en 9.5 cm
    centro del TAMBOR GIRATORIO a 9.0 cm del borde trasero
    => laser_x = -0.005 m, medio centimetro POR DETRAS del centro

El `laser_x = 0` venia del 2026-07-30, anotado como «centrado» SIN cinta detras
— exactamente igual que `laser_z`, que al medirse de verdad resulto estar 2 cm
mal y desplazaba el plano de barrido.

Lo destapo una discrepancia de ~2 cm entre lo que leia /scan tras una parada del
collision_monitor (18.9 cm) y lo que el usuario media en el suelo (7-8 cm):

    con laser_x = 0      residuo 2.3 cm  -> FUERA del ruido de medida
    con laser_x = -0.005 residuo 1.4 cm  -> DENTRO (sus dos esquinas ya
                                            difieren 1.0 cm entre si)

✅ Y `laser_y = 0` deja de ser suposicion: medido con cinta sobre los 21.7 cm.

🔴 `base_length` 0.182 -> 0.190. Las DOS estaban anotadas como medidas con cinta
   y con orugas, y difieren 0.8 cm. Se toma la mas reciente porque es la misma
   con la que se midio laser_x: mezclarlas daria un modelo incoherente consigo
   mismo. ⏳ Conviene arbitrarlo con una escuadra.

📝 `robot_radius` NO se toca: hypot(9.5, 10.85) = 14.4 cm contra los 0.145 m
   configurados. 0.8 mm de diferencia.

✅ Verificado tras compilar y desplegar, en el TF vivo del robot:
       base_footprint -> laser  Translation: [-0.005, 0.000, 0.155]
   (antes [0.000, 0.000, 0.155])

File: atriz_rvr_description/urdf/rvr.urdf.xacro (robot description, xacro)
@@ -64,5 +64,11 @@
           centros. Comprobación: 14.8 + 2×3.5 = 21.8 ≈ 21.7 medidos de lado a
           lado. Las orugas ocupan TODO el ancho del robot. -->
-  <xacro:property name="base_length" value="0.182"/>   <!-- X, frente-atrás   ✅ medido -->
+  <!-- 🔴 0.190 desde el 2026-08-02, no 0.182. Las DOS estaban anotadas como
+       medidas con cinta y con orugas, y difieren 0.8 cm; se toma la mas reciente,
+       que es la misma con la que se midio `laser_x` — mezclarlas daria un modelo
+       incoherente consigo mismo. ⏳ Conviene arbitrarlo con una escuadra.
+       📝 No cambia `robot_radius`: hypot(9.5, 10.85) = 14.4 cm contra los
+          0.145 m configurados. 0.8 mm. -->
+  <xacro:property name="base_length" value="0.190"/>   <!-- X, frente-atrás   ✅ medido 2026-08-02 -->
   <xacro:property name="base_width"  value="0.217"/>   <!-- Y, lado a lado    ✅ medido -->
   <xacro:property name="base_height" value="0.070"/>   <!-- Z, suelo a la tapa ✅ medido -->
@@ -101,6 +107,18 @@
              no afecta a SLAM 2D ni a Nav2, que trabajan en el plano. Afecta a la
              visualización y a ese límite de altura.
-       ✅ CENTRADO y NIVELADO, confirmado por el usuario:
-          · x = 0, y = 0 (2026-07-30)
+       🔴 NO ESTABA CENTRADO EN X. Medido con cinta el 2026-08-02:
+          · chasis 19.0 cm de frente a atras (con orugas) -> centro en 9.5 cm
+          · centro del TAMBOR GIRATORIO a 9.0 cm del borde trasero
+          · => laser_x = -0.005 m, medio centimetro POR DETRAS del centro
+          El «x = 0» de abajo venia del 2026-07-30 y estaba anotado como
+          «centrado» SIN cinta detras — igual que `laser_z`, que al medirse de
+          verdad resulto estar 2 cm mal.
+          📝 Lo destapo una discrepancia de ~2 cm entre lo que leia /scan tras
+             una parada del collision_monitor y lo que el usuario media en el
+             suelo. Con laser_x = 0 el residuo era 2.3 cm (fuera del ruido de
+             medida); con -0.005 baja a 1.4, que ya no se distingue del error
+             de la propia cinta. Evidencia 51.
+       ✅ CENTRADO EN Y y NIVELADO, confirmado por el usuario:
+          · y = 0, medido con cinta sobre los 21.7 cm de ancho (2026-08-02)
           · el disco está a la MISMA altura en los cuatro puntos —delante, detrás,
             izquierda y derecha— (2026-07-31). Es decir: **el robot está físicamente
@@ -108,6 +126,6 @@
             Ver la cabecera de `rvr_driver_node.py` y el manual, cap. 13.
        ═══════════════════════════════════════════════════════════════════════ -->
-  <xacro:property name="laser_x"   value="0.0"/>
-  <xacro:property name="laser_y"   value="0.0"/>
+  <xacro:property name="laser_x"   value="-0.005"/>  <!-- ✅ medido 2026-08-02 -->
+  <xacro:property name="laser_y"   value="0.0"/>     <!-- ✅ medido 2026-08-02 -->
   <xacro:property name="laser_gap" value="0.046"/>   <!-- tapa → base del LIDAR ✅ -->
   <xacro:property name="x2_height" value="0.050"/>   <!-- alto del X2 ✅ medido -->
